File: PCB/IMU_sensor_demo.kicad_pcb (KiCad board)
At the start: 4 copper layers, 0 parts

Commit message: production run for RevA of demo board
Parts:
- added C101: 47u, Capacitor_SMD:C_0805_2012Metric, F.Cu at (130.2, 51.4)
- added C102: 47u, Capacitor_SMD:C_0805_2012Metric, F.Cu at (151.5, 45.0)
- added C103: 47u, Capacitor_SMD:C_0805_2012Metric, F.Cu at (215.2, 45.6)
- added C104: 100n, 0_my_capacitors:C_1005_(0402), F.Cu at (154.7, 46.3)
- added D101: 0603_LED_Red, LED_SMD:LED_0603_1608Metric, F.Cu at (156.5, 60.0)
- added D102: 0603_LED_Red, LED_SMD:LED_0603_1608Metric, F.Cu at (121.5, 95.0)
- added D103: 0603_LED_Red, LED_SMD:LED_0603_1608Metric, F.Cu at (156.5, 70.0)
- added D104: 0603_LED_Red, LED_SMD:LED_0603_1608Metric, F.Cu at (131.5, 95.0)
- added D105: 0603_LED_Red, LED_SMD:LED_0603_1608Metric, F.Cu at (156.5, 80.0)
- added D106: 0603_LED_Red, LED_SMD:LED_0603_1608Metric, F.Cu at (141.5, 95.0)
- added D107: 0603_LED_Red, LED_SMD:LED_0603_1608Metric, F.Cu at (156.5, 90.0)
- added D108: 0603_LED_Red, LED_SMD:LED_0603_1608Metric, F.Cu at (151.5, 95.0)
- added D109: 0603_LED_Red, LED_SMD:LED_0603_1608Metric, F.Cu at (156.5, 100.0)
- added D110: 0603_LED_Red, LED_SMD:LED_0603_1608Metric, F.Cu at (161.5, 95.0)
- added D111: 0603_LED_Red, LED_SMD:LED_0603_1608Metric, F.Cu at (156.5, 110.0)
- added D112: 0603_LED_Red, LED_SMD:LED_0603_1608Metric, F.Cu at (171.5, 95.0)
- added D113: 0603_LED_Red, LED_SMD:LED_0603_1608Metric, F.Cu at (156.5, 120.0)
- added D114: 0603_LED_Red, LED_SMD:LED_0603_1608Metric, F.Cu at (181.5, 95.0)
- added D115: 0603_LED_Red, LED_SMD:LED_0603_1608Metric, F.Cu at (156.5, 130.0)
- added D116: 0603_LED_Red, LED_SMD:LED_0603_1608Metric, F.Cu at (191.5, 95.0)
- added G***: LOGO, 0_my:semify_big, F.Cu at (90.0, 51.0)
- added H101: MountingHole, MountingHole:MountingHole_2.2mm_M2_ISO7380_Pad, F.Cu at (81.5, 40.0)
- added H102: MountingHole, MountingHole:MountingHole_2.2mm_M2_ISO7380_Pad, F.Cu at (81.5, 130.0)
- added H103: MountingHole, MountingHole:MountingHole_2.2mm_M2_ISO7380_Pad, F.Cu at (231.5, 130.0)
- added H104: MountingHole, MountingHole:MountingHole_2.2mm_M2_ISO7380_Pad, F.Cu at (231.5, 40.0)
- added J101: Conn_02x06_Odd_Even, 0_my:PinHeader_2x06_P2.54mm_Horizontal_less_silk, F.Cu at (150.2, 41.1)
- added J102: Conn_01x04_f, Connector_PinSocket_2.54mm:PinSocket_1x04_P2.54mm_Vertical, F.Cu at (214.2, 42.4)
- added JP101: Jumper_2, 0_my:SolderJumper-2_P1.3mm_Bridged, B.Cu at (125.5, 47.5)
- added JP102: Jumper_2, 0_my:SolderJumper-2_P1.3mm_Bridged, B.Cu at (174.0, 51.5)
- added JP103: Jumper_3, 0_my:SolderJumper-3, B.Cu at (178.0, 45.0)
- added R101: 680R, 0_my:R_1005_(0402), F.Cu at (154.7, 47.4)
- added R102: 680R, 0_my:R_1005_(0402), F.Cu at (159.5, 60.0)
- added R103: 680R, 0_my:R_1005_(0402), F.Cu at (121.5, 98.0)
- added R104: 680R, 0_my:R_1005_(0402), F.Cu at (159.5, 70.0)
- added R105: 680R, 0_my:R_1005_(0402), F.Cu at (131.5, 98.0)
- added R106: 680R, 0_my:R_1005_(0402), F.Cu at (159.5, 80.0)
- added R107: 680R, 0_my:R_1005_(0402), F.Cu at (141.5, 98.0)
- added R108: 680R, 0_my:R_1005_(0402), F.Cu at (159.5, 90.0)
- added R109: 680R, 0_my:R_1005_(0402), F.Cu at (151.5, 98.0)
- added R110: 680R, 0_my:R_1005_(0402), F.Cu at (159.5, 100.0)
- added R111: 680R, 0_my:R_1005_(0402), F.Cu at (161.5, 98.0)
- added R112: 680R, 0_my:R_1005_(0402), F.Cu at (159.5, 110.0)
- added R113: 680R, 0_my:R_1005_(0402), F.Cu at (171.5, 98.0)
- added R114: 680R, 0_my:R_1005_(0402), F.Cu at (159.5, 120.0)
- added R115: 680R, 0_my:R_1005_(0402), F.Cu at (181.5, 98.0)
- added R116: 680R, 0_my:R_1005_(0402), F.Cu at (159.5, 130.0)
- added R117: 680R, 0_my:R_1005_(0402), F.Cu at (191.5, 98.0)
- added SW101: Switch, Button_Switch_SMD:SW_SPST_PTS645, F.Cu at (201.5, 75.0)
- added U101: PCF8575_Module, 0_my:PCF8575_Module, F.Cu at (133.7, 42.4)
- added U102: MKI243A_Module, 0_my:STEVAL-MKI243A_Module, F.Cu at (173.0, 54.6)
Routing:
- net +3V3: track 0.00 -> 287.8 mm
- net GND: track 0.00 -> 182.1 mm
- net /p7: track 0.00 -> 127.3 mm
- net /p6: track 0.00 -> 120.9 mm
- net /p5: track 0.00 -> 114.7 mm
- net /p4: track 0.00 -> 108.8 mm
- net /p17: track 0.00 -> 94.0 mm, vias 0 -> 1
- net /p16: track 0.00 -> 86.8 mm, vias 0 -> 1
- net /p15: track 0.00 -> 79.8 mm, vias 0 -> 1
- net /p3: track 0.00 -> 75.9 mm
- net /button: track 0.00 -> 75.0 mm
- net /p14: track 0.00 -> 72.9 mm, vias 0 -> 1
- net /sda: track 0.00 -> 71.2 mm
- net /scl: track 0.00 -> 70.9 mm
- net /p2: track 0.00 -> 67.6 mm
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Other:
- board outline added: 160 x 100 mm
- copper layers 4 -> 2
- board text added: "GND"
- board text added: "PCF8575"
- board text added: "STEVAL-MKI243A ASM330LHHXG1"
- board text added: "VDD"
