File: PCB/IMU_sensor_demo.kicad_sch (KiCad schematic)
At the start: 16 parts, among them J105 STEMMA QT, J106 Conn_02x04, J111 Conn_01x04_f, SW101 Switch

Commit message: production run for RevA of demo board
Parts:
- removed C114, C115: 47u, Capacitor_SMD:C_0805_2012Metric, symbol Device:C_Small
- removed J105: STEMMA QT, Connector_JST:JST_SH_SM04B-SRSS-TB_1x04-1MP_P1.00mm_Horizontal, symbol Connector_Generic_MountingPin:Conn_01x04_MountingPin
- removed J106: Conn_02x04, Connector_PinHeader_2.54mm:PinHeader_2x04_P2.54mm_Vertical, symbol Connector_Generic:Conn_02x04_Odd_Even
- removed R101: 22k, 0_my:R_1005_(0402), symbol Device:R_Small
- added C102, C103: 47u, Capacitor_SMD:C_0805_2012Metric, symbol Device:C_Small
- added D101, D102, D103, D104, D106, D107, D108, D109, D110, D111, D112, D113, D114, D115, D116: 0603_LED_Red, LED_SMD:LED_0603_1608Metric, symbol Device:LED
- added J101: Conn_02x06_Odd_Even, 0_my:PinHeader_2x06_P2.54mm_Horizontal_less_silk, symbol Connector_Generic:Conn_02x06_Odd_Even
- added JP101, JP102: Jumper_2, 0_my:SolderJumper-2_P1.3mm_Bridged, symbol Jumper:Jumper_2_Bridged
- added JP103: Jumper_3, 0_my:SolderJumper-3, symbol Jumper:SolderJumper_3_Bridged12
- added R102, R103, R104, R105, R106, R107, R108, R109, R110, R111, R112, R114, R115, R116, R117: 2k, 0_my:R_1005_(0402), symbol Device:R_Small
- added U101: PCF8575_Module, 0_my:PCF8575_Module, symbol _my:PCF8575_Module
- added U102: MKI243A_Module, 0_my:STEVAL-MKI243A_Module, symbol _my:STEVAL-MKI243A_Module
- D105: value 0603_LED_Yellow -> 0603_LED_Red; LCSC Part # C72038 -> C2286
- J102: renamed from J111; LCSC Part # C2685089 -> C2718488
- R101: renamed from R103; value 13k3 -> 2k; LCSC Part # C274352 -> C4109
- R113: value 5k1 -> 2k; LCSC Part # C105872 -> C4109
- SW101: footprint 0_my:SW_SPST_TS-1088-AR02016 -> Button_Switch_SMD:SW_SPST_PTS645; LCSC Part # C720477 -> C5127964
- renumbered C109 to C104
Connections:
- net +3V3: now also C101.1, R113.1, C102.1, C103.1, J101.1 (Pin_1), J101.2 (Pin_2), JP101.1 (A), JP102.1 (A), JP103.3 (B), R102.1, R103.1, R104.1, R105.1, R106.1, R107.1, R108.1, R109.1, R110.1, R111.1, R112.1, R114.1, R115.1, R116.1, R117.1, U101.4 (VCC), U102.1 (VDD)
- net GND: now also C101.2, C102.2, C103.2, J101.3 (Pin_3), J101.4 (Pin_4), JP103.1 (A), U101.15 (GND), U101.25 (GND), U101.5 (GND), U102.13 (GND)
- net scl: now also J101.7 (Pin_7), U102.20 (SCL)
- net sda: now also J101.9 (Pin_9), U102.21 (SDA)
- net at R113.2: now also D112.2 (A)
- net p2: now reaches D105.1 (K)
- net p2: now also U101.11 (P2)
- net at D105.2 (A): now also R106.2
- net reset_n renamed button
- net button: now also J101.5 (Pin_5)
- new net: D104.2 (A), R105.2
- new net: D108.2 (A), R109.2
- new net: D115.2 (A), R116.2
- new net: D116.2 (A), R117.2
- new net: D103.2 (A), R104.2
- new net: D111.2 (A), R112.2
- new net: D106.2 (A), R107.2
- new net: D110.2 (A), R111.2
- new net: D113.2 (A), R114.2
- new net: D114.2 (A), R115.2
- new net: D107.2 (A), R108.2
- new net: D101.2 (A), R102.2
- new net: D109.2 (A), R110.2
- new net: D102.2 (A), R103.2
- new net cs: U102.19 (CS)
- new net imu_int1: J101.12 (Pin_12), U102.14 (INT1)
- new net imu_int2: J101.11 (Pin_11), U102.15 (INT2)
- new net imu_sdo: JP103.2 (C), U102.22 (SDO)
- new net mscl: U102.4 (MSCL)
- new net msda: U102.5 (MSDA)
- new net p0: D101.1 (K), U101.13 (P0)
- new net p1: D103.1 (K), U101.12 (P1)
- new net p10: D102.1 (K), U101.16 (P10)
- new net p11: D104.1 (K), U101.17 (P11)
- new net p12: D106.1 (K), U101.18 (P12)
- new net p13: D108.1 (K), U101.19 (P13)
- new net p14: D110.1 (K), U101.20 (P14)
- new net p15: D112.1 (K), U101.21 (P15)
- new net p16: D114.1 (K), U101.22 (P16)
- new net p17: D116.1 (K), U101.23 (P17)
- new net p3: D107.1 (K), U101.10 (P3)
- new net p4: D109.1 (K), U101.9 (P4)
- new net p5: D111.1 (K), U101.8 (P5)
- new net p6: D113.1 (K), U101.7 (P6)
- new net p7: D115.1 (K), U101.6 (P7)
- new net pcf_int_n: J101.10 (Pin_10), U101.1 (~{INT})
- new net scl2: J101.8 (Pin_8), U101.2 (SCL)
- new net sda2: J101.6 (Pin_6), U101.3 (SDA)
- new net vdd: JP101.2 (B), U101.14 (VDD), U101.24 (VDD)
- new net vdd_io: JP102.2 (B), U102.2 (VDD_IO)
Other:
- note added: "Button"
- note added: "IMU Sensor"
- note added: "PCF8575"
- note added: "PMOD"
- note removed: "i2c headers"
- moved on the sheet: C104, J102, R101, SW101
